File: Electronic/schematics.kicad_sch (KiCad schematic)
At the start: 28 parts, among them J1 Jack-DC, J2 Conn_01x04_Socket, J3 Conn_01x03, U1 ESP32-S3-DEVKITC-1-N16R8V, U2 TMC2209_SILENTSTEPSTICK, U3 DC-DC 12V-3V buck, U4 74HC14

Commit message: Refactor schematics and update PCB images
- Removed unconnected items from the KiCad project file.
- Removed a diode symbol (PESD3V3S1UL) and its associated properties from the schematic.
- Renamed and repositioned several pins in the TMC2209_SILENTSTEPSTICK symbol for clarity.
- Cleaned up unnecessary junctions and wires in the schematic.
- Updated multiple PCB and schematic images to reflect recent design changes.
Parts:
- removed D2, D3, D4: PESD3V3S1UL, Diode_SMD:D_SOD-882, symbol Diode:PESD3V3S1UL
Connections:
- net at R1.2, U1.11 (GPIO18): now also U2.13 (UART); no longer U2.12 (UART)
